File: Schematics/Control Board/mega_pro-v13/frc_operator_interface.sch (EAGLE design)
At the start: 47 parts, among them CN1 1uF, CN2 1uF, CN3 1uF, CN4 1uF, J1 AVR_SPI_PRG_6PTH, U1 TLC59282_DBQ_24, U4 FT232RLSSOP, Y1 RESONATORSMD

Commit message: Final control board revision 1.1
Parts:
- removed C10, C30: 10uF, rcl:C-USC1206
- removed C9: 0.1uF, rcl:C-USC1206
- removed R4, R5: 10k, rcl:R-US_M1206
- removed U$15: I2CHEADER, teamFusion:I2CHEADER
Connections:
- net 5V: no longer C10.1, C30.1, C9.1, R4.2, R5.2, U$15.VCC
- net DIO20(SDA): no longer R5.1, U$15.SDA
- net DIO21(SCL): no longer R4.1, U$15.SCL
- net GND: no longer C10.2, C30.2, C9.2, U$15.GND
Changed lines of the file:
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@@
 <part name="C7" library="rcl" deviceset="C-US" device="C1206" value="0.1uF"/>
 <part name="C8" library="rcl" deviceset="C-US" device="C1206" value="0.1uF"/>
-<part name="R4" library="rcl" deviceset="R-US_" device="M1206" value="10k"/>
-<part name="R5" library="rcl" deviceset="R-US_" device="M1206" value="10k"/>
 <part name="R6" library="rcl" deviceset="R-US_" device="M1206" value="170"/>
 <part name="POWER" library="SparkFun-LED" deviceset="LED" device="3MM"/>
@@
 <part name="GND13" library="SparkFun" deviceset="GND" device=""/>
 <part name="RESET" library="switch-omron" deviceset="10-XX" device=""/>
-<part name="C9" library="rcl" deviceset="C-US" device="C1206" value="0.1uF"/>
-<part name="C10" library="rcl" deviceset="C-US" device="C1206" value="10uF"/>
 <part name="GND15" library="SparkFun" deviceset="GND" device=""/>
 <part name="GND16" library="SparkFun" deviceset="GND" device=""/>
 <part name="U4" library="SparkFun" deviceset="FT232RL" device="SSOP"/>
-<part name="GND17" library="SparkFun" deviceset="GND" device=""/>
-<part name="GND18" library="SparkFun" deviceset="GND" device=""/>
 <part name="R1" library="rcl" deviceset="R-US_" device="M1206" value="280"/>
 <part name="R2" library="rcl" deviceset="R-US_" device="M1206" value="315"/>
@@
 <part name="U$13" library="SparkFun" deviceset="5V" device=""/>
 <part name="U$14" library="teamFusion" deviceset="UE27BC54130-USB" device=""/>
-<part name="U$15" library="teamFusion" deviceset="I2CHEADER" device=""/>
-<part name="C30" library="rcl" deviceset="C-US" device="C1206" value="10uF"/>
 <part name="C31" library="rcl" deviceset="C-US" device="C1206" value="10uF"/>
 <part name="C32" library="rcl" deviceset="C-US" device="C1206" value="10uF"/>
@@
 <part name="U$2" library="teamFusion" deviceset="DIGITALIN" device=""/>
 <part name="GND1" library="SparkFun" deviceset="GND" device=""/>
-<part name="U$9" library="SparkFun" deviceset="5V" device=""/>
 <part name="C1" library="rcl" deviceset="C-US" device="C1206" value="0.1uF"/>
 <part name="GND5" library="SparkFun" deviceset="GND" device=""/>
@@
 <instance part="C7" gate="G$1" x="213.36" y="162.56"/>
 <instance part="C8" gate="G$1" x="205.74" y="162.56"/>
-<instance part="R4" gate="G$1" x="58.42" y="40.64"/>
-<instance part="R5" gate="G$1" x="58.42" y="30.48"/>
 <instance part="R6" gate="G$1" x="124.46" y="218.44" rot="R90"/>
 <instance part="POWER" gate="G$1" x="124.46" y="208.28"/>
@@
 <instance part="GND13" gate="1" x="337.82" y="149.86"/>
 <instance part="RESET" gate="1" x="200.66" y="195.58"/>
-<instance part="C9" gate="G$1" x="33.02" y="160.02"/>
-<instance part="C10" gate="G$1" x="43.18" y="160.02"/>
 <instance part="GND15" gate="1" x="73.66" y="134.62"/>
 <instance part="GND16" gate="1" x="12.7" y="187.96" rot="R180"/>
 <instance part="U4" gate="G$1" x="91.44" y="157.48"/>
-<instance part="GND17" gate="1" x="33.02" y="149.86"/>
-<instance part="GND18" gate="1" x="43.18" y="149.86"/>
 <instance part="R1" gate="G$1" x="147.32" y="167.64" rot="R90"/>
 <instance part="R2" gate="G$1" x="154.94" y="167.64" rot="R90"/>
@@
 <instance part="U$13" gate="G$1" x="144.78" y="5.08"/>
 <instance part="U$14" gate="G$1" x="-2.54" y="175.26"/>
-<instance part="U$15" gate="G$1" x="20.32" y="43.18"/>
-<instance part="C30" gate="G$1" x="66.04" y="50.8" rot="R180"/>
 <instance part="C31" gate="G$1" x="152.4" y="-20.32"/>
 <instance part="C32" gate="G$1" x="139.7" y="127"/>
@@
 <instance part="U$2" gate="G$1" x="226.06" y="-15.24"/>
 <instance part="GND1" gate="1" x="210.82" y="-40.64"/>
-<instance part="U$9" gate="G$1" x="78.74" y="48.26"/>
 <instance part="C1" gate="G$1" x="53.34" y="160.02"/>
 <instance part="GND5" gate="1" x="53.34" y="149.86"/>
@@
 <pinref part="U4" gate="G$1" pin="GND21"/>
 <pinref part="GND15" gate="1" pin="GND"/>
-</segment>
-<segment>
-<pinref part="C9" gate="G$1" pin="2"/>
-<pinref part="GND17" gate="1" pin="GND"/>
-<wire x1="33.02" y1="154.94" x2="33.02" y2="152.4" width="0.1524" layer="91"/>
-</segment>
-<segment>
-<wire x1="43.18" y1="152.4" x2="43.18" y2="154.94" width="0.1524" layer="91"/>
-<pinref part="C10" gate="G$1" pin="2"/>
-<pinref part="GND18" gate="1" pin="GND"/>
 </segment>
 <segment>
@@
 </segment>
 <segment>
-<pinref part="U$15" gate="G$1" pin="GND"/>
-<wire x1="38.1" y1="48.26" x2="53.34" y2="48.26" width="0.1524" layer="91"/>
-<label x="35.56" y="48.26" size="1.778" layer="95"/>
-<wire x1="53.34" y1="48.26" x2="53.34" y2="58.42" width="0.1524" layer="91"/>
-<wire x1="53.34" y1="58.42" x2="66.04" y2="58.42" width="0.1524" layer="91"/>
-<pinref part="C30" gate="G$1" pin="2"/>
-<wire x1="66.04" y1="58.42" x2="66.04" y2="55.88" width="0.1524" layer="91"/>
-</segment>
-<segment>
 <pinref part="U$2" gate="G$1" pin="GND"/>
 <pinref part="GND1" gate="1" pin="GND"/>
@@
 <pinref part="GND" gate="1" pin="(SCL/INT0)PD0"/>
 </segment>
-<segment>
-<pinref part="U$15" gate="G$1" pin="SCL"/>
-<wire x1="38.1" y1="43.18" x2="50.8" y2="43.18" width="0.1524" layer="91"/>
-<label x="35.56" y="43.18" size="1.778" layer="95"/>
-<wire x1="50.8" y1="43.18" x2="50.8" y2="40.64" width="0.1524" layer="91"/>
-<pinref part="R4" gate="G$1" pin="1"/>
-<wire x1="50.8" y1="40.64" x2="53.34" y2="40.64" width="0.1524" layer="91"/>
-</segment>
 </net>
 <net name="DIO20(SDA)" class="0">
@@
 <label x="314.96" y="119.38" size="1.778" layer="95"/>
 <pinref part="GND" gate="1" pin="(SDA/INT1)PD1"/>
-</segment>
-<segment>
-<pinref part="U$15" gate="G$1" pin="SDA"/>
-<wire x1="38.1" y1="40.64" x2="43.18" y2="40.64" width="0.1524" layer="91"/>
-<label x="35.56" y="40.64" size="1.778" layer="95"/>
-<wire x1="43.18" y1="40.64" x2="43.18" y2="30.48" width="0.1524" layer="91"/>
-<pinref part="R5" gate="G$1" pin="1"/>
-<wire x1="43.18" y1="30.48" x2="53.34" y2="30.48" width="0.1524" layer="91"/>
 </segment>
 </net>
@@
 <net name="5V" class="1">
 <segment>
-<wire x1="33.02" y1="177.8" x2="43.18" y2="177.8" width="0.1524" layer="91"/>
-<wire x1="43.18" y1="177.8" x2="60.96" y2="177.8" width="0.1524" layer="91"/>
+<wire x1="27.94" y1="177.8" x2="60.96" y2="177.8" width="0.1524" layer="91"/>
 <wire x1="60.96" y1="177.8" x2="60.96" y2="167.64" width="0.1524" layer="91"/>
 <wire x1="60.96" y1="167.64" x2="76.2" y2="167.64" width="0.1524" layer="91"/>
-<wire x1="43.18" y1="162.56" x2="43.18" y2="177.8" width="0.1524" layer="91"/>
-<wire x1="33.02" y1="162.56" x2="33.02" y2="177.8" width="0.1524" layer="91"/>
 <wire x1="60.96" y1="180.34" x2="60.96" y2="177.8" width="0.1524" layer="91"/>
-<junction x="43.18" y="177.8"/>
 <junction x="60.96" y="177.8"/>
 <pinref part="U4" gate="G$1" pin="VCC"/>
-<pinref part="C10" gate="G$1" pin="1"/>
-<pinref part="C9" gate="G$1" pin="1"/>
 <pinref part="U$4" gate="G$1" pin="5V"/>
 <pinref part="F1" gate="G$1" pin="2"/>
-<wire x1="27.94" y1="177.8" x2="33.02" y2="177.8" width="0.1524" layer="91"/>
-<junction x="33.02" y="177.8"/>
 <pinref part="U4" gate="G$1" pin="VCCIO"/>
 <wire x1="76.2" y1="162.56" x2="60.96" y2="162.56" width="0.1524" layer="91"/>
@@
 </segment>
 <segment>
-<wire x1="63.5" y1="40.64" x2="66.04" y2="40.64" width="0.1524" layer="91"/>
-<wire x1="66.04" y1="40.64" x2="66.04" y2="30.48" width="0.1524" layer="91"/>
-<wire x1="66.04" y1="30.48" x2="63.5" y2="30.48" width="0.1524" layer="91"/>
-<wire x1="66.04" y1="48.26" x2="66.04" y2="45.72" width="0.1524" layer="91"/>
-<junction x="66.04" y="40.64"/>
-<pinref part="R4" gate="G$1" pin="2"/>
-<pinref part="R5" gate="G$1" pin="2"/>
-<pinref part="C30" gate="G$1" pin="1"/>
-<pinref part="U$15" gate="G$1" pin="VCC"/>
-<wire x1="66.04" y1="45.72" x2="66.04" y2="40.64" width="0.1524" layer="91"/>
-<wire x1="38.1" y1="45.72" x2="66.04" y2="45.72" width="0.1524" layer="91"/>
-<wire x1="66.04" y1="45.72" x2="78.74" y2="45.72" width="0.1524" layer="91"/>
-<junction x="66.04" y="45.72"/>
-<pinref part="U$9" gate="G$1" pin="5V"/>
-<wire x1="78.74" y1="45.72" x2="78.74" y2="48.26" width="0.1524" layer="91"/>
-</segment>
-<segment>
