File: Projects/FRC Operator Interface Control Board/controlBoard_EagleProject/frc_operator_interface.brd (EAGLE design)
At the start: 99.1 x 99.1 mm, 41 parts, among them CN1 1uF, CN2 1uF, CN3 1uF, CN4 1uF, J1 AVR_SPI_PRG_6PTH, J2 ANALOGHEADER, J3 DIGITALIN, J4 DIGITALOUTPUTS, J5 PWMHEADER, J6 UE27BC54130-USB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

Commit message: Updated the resistor values for some of the LEDs on the board. Controller board code update commit.
Parts:
- removed R1: 280, rcl:M1206
- removed R2: 315, rcl:M1206
- R6: value 170 -> 1.8k
- R7: value 300 -> 330
Connections:
- removed net N$1: R1.1, TX.A
- removed net N$5: R2.1, RX.A
- net 5V: now also RX.A, TX.A; no longer R1.2, R2.2
Routing:
- net N$5: track 2.41 -> 0.00 mm
- net N$1: track 2.41 -> 0.00 mm
- net 5V: track 245.2 -> 244.4 mm, vias 15 -> 13
Other:
- board text added: "Revision 1.2"
- board text removed: "Revision 1.1"
Changed lines of the file:
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@@
 <?xml version="1.0" encoding="utf-8"?>
 <!DOCTYPE eagle SYSTEM "eagle.dtd">
-<eagle version="6.5.0">
+<eagle version="7.5.0">
 <drawing>
 <settings>
@@
 <layer number="59" name="tCarbon" color="7" fill="1" visible="no" active="no"/>
 <layer number="60" name="bCarbon" color="7" fill="1" visible="no" active="no"/>
-<layer number="90" name="Modules" color="5" fill="1" visible="no" active="yes"/>
+<layer number="90" name="Modules" color="5" fill="1" visible="no" active="no"/>
 <layer number="91" name="Nets" color="2" fill="1" visible="no" active="no"/>
 <layer number="92" name="Busses" color="1" fill="1" visible="no" active="no"/>
@@
 <text x="47.117" y="69.215" size="2.54" layer="25" ratio="16">Designed by:</text>
 <text x="47.117" y="65.405" size="2.54" layer="25" ratio="16">Ryan Nazaretian</text>
-<text x="47.117" y="61.595" size="2.54" layer="25" ratio="16">Revision 1.1</text>
+<text x="47.117" y="61.595" size="2.54" layer="25" ratio="16">Revision 1.2</text>
 </plain>
 <attributes>
@@
 <pass name="Default">
 <param name="RoutingGrid" value="50mil"/>
+<param name="AutoGrid" value="1"/>
+<param name="Efforts" value="0"/>
+<param name="TopRouterVariant" value="1"/>
 <param name="tpViaShape" value="round"/>
 <param name="PrefDir.1" value="|"/>
@@
 <element name="C7" library="rcl" package="C1206" value="0.1uF" x="53.7845" y="23.33625" rot="R270"/>
 <element name="C8" library="rcl" package="C1206" value="0.1uF" x="42.926" y="43.434" rot="R90"/>
-<element name="R6" library="rcl" package="M1206" value="170" x="26.797" y="82.55" rot="R270"/>
+<element name="R6" library="rcl" package="M1206" value="1.8k" x="26.797" y="82.55" rot="R270"/>
 <element name="POWER" library="SparkFun-LED" package="LED3MM" value="" x="26.797" y="87.63" rot="R90"/>
-<element name="R7" library="rcl" package="M1206" value="300" x="9.652" y="82.55" rot="R270"/>
+<element name="R7" library="rcl" package="M1206" value="330" x="9.652" y="82.55" rot="R270"/>
 <element name="STATUS" library="SparkFun-LED" package="LED3MM" value="" x="9.652" y="87.63" rot="R90"/>
 <element name="RESET" library="switch-omron" package="B3F-10XX" value="" x="24.638" y="59.944" rot="R270">
@@
 </element>
 <element name="U2" library="SparkFun" package="SSOP28DB" value="FT232RLSSOP" x="27.051" y="70.358" rot="R90"/>
-<element name="R1" library="rcl" package="M1206" value="280" x="21.082" y="82.55" rot="R270"/>
-<element name="R2" library="rcl" package="M1206" value="315" x="15.367" y="82.55" rot="R270"/>
 <element name="TX" library="SparkFun-LED" package="LED3MM" value="" x="21.082" y="87.63" rot="R90"/>
 <element name="RX" library="SparkFun-LED" package="LED3MM" value="" x="15.367" y="87.63" rot="R90"/>
@@
 <wire x1="25.146" y1="75.819" x2="22.352" y2="78.613" width="0.254" layer="1"/>
 </signal>
-<signal name="N$1">
-<contactref element="R1" pad="1"/>
-<contactref element="TX" pad="A"/>
-<wire x1="21.082" y1="86.36" x2="21.082" y2="83.95" width="0.4064" layer="1"/>
-</signal>
-<signal name="N$5">
-<contactref element="R2" pad="1"/>
-<contactref element="RX" pad="A"/>
-<wire x1="15.367" y1="86.36" x2="15.367" y2="83.95" width="0.4064" layer="1"/>
-</signal>
 <signal name="TXD">
 <contactref element="U2" pad="1"/>
@@
 <signal name="5V" class="1">
 <contactref element="U2" pad="20"/>
-<contactref element="R1" pad="2"/>
-<contactref element="R2" pad="2"/>
 <contactref element="R6" pad="2"/>
 <contactref element="R3" pad="2"/>
@@
 <wire x1="50.577" y1="35.21" x2="50.927" y2="35.56" width="0.254" layer="1"/>
 <wire x1="50.927" y1="35.56" x2="50.927" y2="37.335" width="0.254" layer="1"/>
-<via x="21.082" y="80.9625" extent="1-16" drill="0.3048"/>
 <via x="26.797" y="80.9625" extent="1-16" drill="0.3048"/>
-<wire x1="21.082" y1="80.9625" x2="21.082" y2="81.15" width="0.254" layer="1"/>
 <wire x1="26.797" y1="80.9625" x2="26.797" y2="81.15" width="0.254" layer="1"/>
 <wire x1="42.902" y1="37.21" x2="42.902" y2="41.756" width="0.254" layer="1"/>
@@
 <via x="41.81475" y="17.43075" extent="1-16" drill="0.3048"/>
 <wire x1="18.44675" y1="62.38875" x2="18.542" y2="62.484" width="0.6096" layer="1"/>
-<via x="15.367" y="81.12125" extent="1-16" drill="0.3048"/>
 <via x="29.0195" y="68.10375" extent="1-16" drill="0.3048"/>
 <wire x1="30.707" y1="68.083" x2="29.04025" y2="68.083" width="0.254" layer="1"/>
@@
 <wire x1="28.702" y1="35.56" x2="28.321" y2="35.684" width="0.254" layer="1"/>
 <wire x1="17.272" y1="81.28" x2="16.002" y2="82.55" width="0.254" layer="16"/>
-<wire x1="16.002" y1="81.28" x2="15.367" y2="81.15" width="0.254" layer="1"/>
 <wire x1="84.328" y1="73.66" x2="84.84535" y2="73.6092" width="0.254" layer="1"/>
 <wire x1="41.711659375" y1="17.44575625" x2="41.16474375" y2="17.44575625" width="0.254" layer="1"/>
@@
 <wire x1="40.402" y1="18.120415625" x2="41.076659375" y2="17.44575625" width="0.254" layer="1"/>
 <wire x1="41.076659375" y1="17.44575625" x2="41.711659375" y2="17.44575625" width="0.254" layer="1"/>
-<wire x1="15.367" y1="81.15" x2="15.367" y2="81.12125" width="0.254" layer="1"/>
 <wire x1="84.84535" y1="73.6092" x2="85.0138" y2="73.6092" width="0.254" layer="1"/>
 <wire x1="20.066" y1="69.596" x2="21.803" y2="71.333" width="0.254" layer="1"/>
@@
 <wire x1="35.052" y1="83.82" x2="37.592" y2="83.82" width="1.6764" layer="1"/>
 <wire x1="35.052" y1="83.82" x2="32.512" y2="83.82" width="1.6764" layer="1"/>
+<contactref element="TX" pad="A"/>
+<contactref element="RX" pad="A"/>
+<wire x1="73.152" y1="82.677" x2="84.328" y2="73.66" width="0" layer="19" extent="1-1"/>
+<wire x1="26.797" y1="81.15" x2="32.512" y2="83.82" width="0" layer="19" extent="1-16"/>
+<wire x1="19.812" y1="81.7" x2="26.797" y2="81.15" width="0" layer="19" extent="1-16"/>
+<wire x1="15.367" y1="86.36" x2="16.002" y2="82.55" width="0" layer="19" extent="16-16"/>
+<wire x1="21.082" y1="86.36" x2="19.812" y2="81.7" width="0" layer="19" extent="16-16"/>
+<wire x1="23.395" y1="71.333" x2="26.797" y2="80.9625" width="0" layer="19" extent="1-1"/>
+<wire x1="29.0195" y1="68.10375" x2="23.395" y2="71.333" width="0" layer="19" extent="1-1"/>
+<wire x1="10.06475" y1="48.10125" x2="18.8214" y2="60.582" width="0" layer="19" extent="1-1"/>
+<wire x1="10.06475" y1="45.56125" x2="10.06475" y2="48.10125" width="0" layer="19" extent="1-1"/>
+<wire x1="10.06475" y1="43.02125" x2="10.06475" y2="45.56125" width="0" layer="19" extent="1-1"/>
+<wire x1="10.06475" y1="40.48125" x2="10.06475" y2="43.02125" width="0" layer="19" extent="1-1"/>
+<wire x1="10.06475" y1="37.94125" x2="10.06475" y2="40.48125" width="0" layer="19" extent="1-1"/>
+<wire x1="10.06475" y1="35.40125" x2="10.06475" y2="37.94125" width="0" layer="19" extent="1-1"/>
+<wire x1="10.06475" y1="32.86125" x2="10.06475" y2="35.40125" width="0" layer="19" extent="1-1"/>
+<wire x1="10.06475" y1="30.32125" x2="10.06475" y2="32.86125" width="0" layer="19" extent="1-1"/>
+<wire x1="10.06475" y1="27.78125" x2="10.06475" y2="30.32125" width="0" layer="19" extent="1-1"/>
+<wire x1="10.06475" y1="25.24125" x2="10.06475" y2="27.78125" width="0" layer="19" extent="1-1"/>
+<wire x1="10.06475" y1="22.70125" x2="10.06475" y2="25.24125" width="0" layer="19" extent="1-1"/>
+<wire x1="10.06475" y1="20.16125" x2="10.06475" y2="22.70125" width="0" layer="19" extent="1-1"/>
+<wire x1="10.06475" y1="17.62125" x2="10.06475" y2="20.16125" width="0" layer="19" extent="1-1"/>
+<wire x1="10.06475" y1="15.08125" x2="10.06475" y2="17.62125" width="0" layer="19" extent="1-1"/>
+<wire x1="10.06475" y1="12.54125" x2="10.06475" y2="10.00125" width="0" layer="19" extent="1-1"/>
+<wire x1="22.45995" y1="26.40965" x2="10.06475" y2="25.24125" width="0" layer="19" extent="1-1"/>
+<wire x1="32.06" y1="32.71" x2="24.511" y2="26.4795" width="0" layer="19" extent="1-1"/>
+<wire x1="42.902" y1="37.21" x2="33.402" y2="32.71" width="0" layer="19" extent="1-1"/>
+<wire x1="47.752" y1="35.21" x2="42.902" y2="37.21" width="0" layer="19" extent="1-16"/>
+<wire x1="49.402" y1="35.21" x2="47.752" y2="35.14" width="0" layer="19" extent="1-16"/>
+<wire x1="49.402" y1="25.21" x2="49.402" y2="35.21" width="0" layer="19" extent="1-1"/>
+<wire x1="40.402" y1="21.21" x2="49.402" y2="25.21" width="0" layer="19" extent="1-1"/>
+<wire x1="26.035" y1="46.99" x2="28.321" y2="35.684" width="0" layer="19" extent="1-1"/>
 </signal>
 <signal name="N$4">
